Commit message: Delta 3-DOF thesis: kinematics, trajectory, pick-and-place
- delta_controller: closed-form IK/FK, min-jerk Cartesian trajectories,
  interactive cartesian_control node, vacuum gripper node (DetachableJoint)
  and pick_place launch file, with unit tests
- delta_objects_world.sdf: table, three objects, drop bin
- 3dof_delta: platform collision + per-object gripper plugins
- CLAUDE.md: project notes and verified results

Co-Authored-By: Claude Opus 5 <noreply@anthropic.com>

File: src/closed_loop_description/urdf/3dof_delta.urdf.xacro (robot description, xacro)
@@ -312,4 +312,14 @@
       </material>
     </visual>
+    <!-- Collision (đồ án): chỉ platform có va chạm để đẩy/chạm vật; cánh tay vẫn không có.
+         Xấp xỉ tấm Werkzeugtraeger (bbox ~0.059 x 0.051 x 0.006 m) bằng hộp dẹt.
+         Hạn chế đã đo: ép platform XUỐNG vật động đang nằm trên bàn thì platform lún dần vào vật
+         (~mm, với cả hộp/trụ/cầu); đẩy ngang và chạm bàn tĩnh thì ổn định. -->
+    <collision>
+      <origin xyz="0 0 0" rpy="0 0 0"/>
+      <geometry>
+        <box size="0.05 0.05 0.006"/>
+      </geometry>
+    </collision>
     <inertial>
       <origin xyz="0 0 0" rpy="0 0 0"/>
@@ -498,4 +508,5 @@
   </joint>
     <xacro:include filename="3dof_delta.gazebo.xacro"/>
+    <xacro:include filename="3dof_delta.gripper.xacro"/>
   </xacro:if>  <!-- end sim: closure helpers + Gazebo plugins -->
   <xacro:if value="$(arg ros2_control)">
