Commit message: Step 10b: cans, three sorting bins, and a highlighted suction head

File: src/closed_loop_description/urdf/3dof_delta.gripper.xacro (robot description, xacro)
@@ -7,6 +7,7 @@
      Plugin (gz-sim8) tự ATTACH ngay khi tìm thấy vật -> gripper_node phải gửi detach cho tất cả
      vật lúc khởi động. World không có vật (delta_world.sdf) thì plugin chỉ chờ, không cảnh báo.
-     Danh sách vật phải khớp với: worlds/delta_objects_world.sdf và
-     delta_controller/launch/pick_place.launch.py (OBJECTS). -->
+     Khai báo vật của CẢ HAI thế giới: ba lon (delta_cans_world.sdf, dùng từ Bước 10b) và ba
+     khối vuông cũ (delta_objects_world.sdf, giữ để tái lập Bước 6–9). Plugin chỉ chờ chứ không
+     cảnh báo khi world không có vật đó (suppress_child_warning), nên khai cả 6 là an toàn. -->
 <robot xmlns:xacro="http://www.ros.org/wiki/xacro">
   <xacro:macro name="vacuum_target" params="object">
@@ -24,4 +25,9 @@
     </gazebo>
   </xacro:macro>
+  <!-- Ba lon (cảnh hiện tại, scene.OBJECTS) -->
+  <xacro:vacuum_target object="coca_can"/>
+  <xacro:vacuum_target object="pepsi_can"/>
+  <xacro:vacuum_target object="sevenup_can"/>
+  <!-- Ba khối vuông của thế giới cũ (scene.LEGACY_OBJECTS) -->
   <xacro:vacuum_target object="red_box"/>
   <xacro:vacuum_target object="green_cylinder"/>

File: src/closed_loop_description/urdf/3dof_delta.urdf.xacro (robot description, xacro)
@@ -311,4 +311,26 @@
         <color rgba="0.95 0.75 0.10 1.0"/>
       </material>
+    </visual>
+    <!-- ĐẦU HÚT (đồ án): hai khối CHỈ HIỂN THỊ, không va chạm, không đổi vật lý — để nhìn rõ đầu
+         công tác đang ở đâu trong mô phỏng và trên ảnh camera.
+         Màu hồng cánh sen (H ≈ 157 trong HSV) nằm NGOÀI cả ba lớp màu đỏ [0,8]∪[172,180],
+         lục [45,85], lam [95,125] nên bộ nhận dạng không coi đầu hút là vật.
+         Mặt hút nằm ÂM trong bề dày platform (z -0.003..0), không thò xuống dưới mặt dưới, để
+         không đâm vào vật khi hạ tới điểm chạm (tool0 z = đỉnh vật + 0.003). -->
+    <visual name="suction_face">
+      <origin xyz="0 0 -0.0015" rpy="0 0 0"/>
+      <geometry>
+        <cylinder radius="0.009" length="0.003"/>
+      </geometry>
+      <material name="mat_suction">
+        <color rgba="1.0 0.10 0.80 1.0"/>
+      </material>
+    </visual>
+    <visual name="suction_turret">
+      <origin xyz="0 0 0.007" rpy="0 0 0"/>
+      <geometry>
+        <cylinder radius="0.010" length="0.008"/>
+      </geometry>
+      <material name="mat_suction"/>
     </visual>
     <!-- Collision (đồ án): chỉ platform có va chạm để đẩy/chạm vật; cánh tay vẫn không có.
